Commit message: ADD:rtabmap mapping

File: omo_r1_description/urdf/omo_r1.urdf.xacro (robot description, xacro)
@@ -160,5 +160,5 @@
   </link>
   <joint name="camera_joint" type="fixed">
-    <origin xyz="0.07 0.0 0.63" rpy="0 0.7 0"/>
+    <origin xyz="0.07 0.0 0.63" rpy="0 0 0"/>
     <parent link="base_link"/>
     <child link="camera_link"/>
@@ -166,5 +166,5 @@
   <link name="camera_link">
     <visual>
-      <origin xyz="0 0 0.0" rpy="1.5758 0.0 1.5758"/>
+      <origin xyz="0 0 0.0" rpy="0 0.0 0"/>
       <geometry>
         <mesh filename="package://omo_r1_description/meshes/sensors/omo_r1_camera.stl" scale="0.001 0.001 0.001"/>

File: omo_r1_gazebo/sdf/omo_r1.gazebo.xacro (robot description, xacro)
@@ -56,5 +56,5 @@
     <plugin name="omo_r1_controller" filename="libgazebo_ros_diff_drive.so">
       <commandTopic>cmd_vel</commandTopic>
-      <odometryTopic>odom</odometryTopic>
+      <odometryTopic>camera/odom</odometryTopic>
       <odometryFrame>odom</odometryFrame>
       <odometrySource>world</odometrySource>
@@ -103,4 +103,49 @@
     </plugin>
   </gazebo>
+  <!-- RGBD Camera -->
+  <gazebo reference="camera_link">
+    <sensor type="depth" name="camera">
+        <always_on>1</always_on>
+        <update_rate>20.0</update_rate>
+        <visualize>true</visualize>
+        <camera>
+            <horizontal_fov>1.047</horizontal_fov>
+            <image>
+                <width>640</width>
+                <height>480</height>
+                <format>R8G8B8</format>
+            </image>
+            <depth_camera>
+            </depth_camera>
+            <clip>
+                <near>0.1</near>
+                <far>20</far>
+            </clip>
+        </camera>
+         <plugin name="camera_plugin" filename="libgazebo_ros_openni_kinect.so">
+            <baseline>0.2</baseline>
+            <alwaysOn>true</alwaysOn>
+            <updateRate>10.0</updateRate>
+            <cameraName>camera</cameraName>
+            <frameName>camera_rgb_optical_frame</frameName>
+            <imageTopicName>rgb/image_raw</imageTopicName>
+            <depthImageTopicName>depth/image_raw</depthImageTopicName>
+            <pointCloudTopicName>depth/points</pointCloudTopicName>
+            <cameraInfoTopicName>rgb/camera_info</cameraInfoTopicName>
+            <depthImageCameraInfoTopicName>depth/camera_info</depthImageCameraInfoTopicName>
+            <pointCloudCutoff>0.4</pointCloudCutoff>
+                <hackBaseline>0.07</hackBaseline>
+                <distortionK1>0.0</distortionK1>
+                <distortionK2>0.0</distortionK2>
+                <distortionK3>0.0</distortionK3>
+                <distortionT1>0.0</distortionT1>
+                <distortionT2>0.0</distortionT2>
+            <CxPrime>0.0</CxPrime>
+            <Cx>0.0</Cx>
+            <Cy>0.0</Cy>
+            <focalLength>0.0</focalLength>
+            </plugin>
+    </sensor>
+  </gazebo>
   <gazebo reference="base_scan">
     <material>Gazebo/FlatBlack</material>
